File: PCB/SensorNode.sch (EAGLE design)
At the start: 54 parts, among them Q1 CMA-4544PF-W, U1 MAX4466EXK+T, U2 ESP-WROOM-32, U3 Si7021-A20, U4 MCP73831, U5 TSL2561, U7 V_REG_317SMD

Commit message: PCB Improvements, layout planned out
Moved components around on layout to minimize pcb space. Battery moved
to back of board. Minor schematic improvements. ESP32 template added
Parts:
- removed C9: 4.7uF, SparkFun-Capacitors:4.7UF-6.3V-10%(0603)0603
- removed D11: RED, SparkFun-LED:LED-RED0603
- added C10: 4.7uF, microbuilder:CAP_CERAMIC0805-NOOUTLINE
- added D4: RED, SparkFun-LED:LED-RED1206
- added R21: 330, microbuilder:RESISTOR0805
- added R22, R23: 10K, adafruit:R-US_R0805
- C8: device SparkFun-Capacitors:4.7UF-6.3V-10%(0603)0603 -> microbuilder:CAP_CERAMIC0805-NOOUTLINE
- R12: value 330 -> 2k; device SparkFun-Resistors:330OHM1/10W1%(0603) -> microbuilder:RESISTOR0805
- R13: value 2.0k -> 10K; device SparkFun-Resistors:2.0KOHM1/10W5%(0603) -> adafruit:R-US_R0805
Connections:
- new net IO23: U2.IO26
- new net IO25: U2.IO25
- new net IO33: U2.IO33
- new net N$35: R13.1, S1.1
- net GND: now also C10.1, C8.1, R12.1; no longer C8.2, C9.2, R13.2
- net N$23: now also D4.A, R21.2; no longer D11.A, R12.1
- net PROG: now also R12.2; no longer R13.1
- net STAT: now also D4.C; no longer D11.C
- net VCC: now also R13.2, R22.2, R23.2; no longer S1.1, S2.1, S3.1
- net VCC_3.7V: now also C8.2; no longer C9.1
- net VIN: now also C10.2, R21.1; no longer C8.1, R12.2
Other:
- moved on the sheet: C8, R13, S1, S2, S3

Commit message: Added USB to UART and Auto Reset Circuit
Parts:
- removed C7: 0.1uF, adafruit:C-USC0805
- removed J3: (no value), SparkFun-Connectors:CONN_06SILK_FEMALE_PTH
- removed R12(NC), R6(NC): 0K, microbuilder:RESISTOR0805
- added C11: 0.1uF, microbuilder:CAP_CERAMIC0805-NOOUTLINE
- added C9: 4.7uF, microbuilder:CAP_CERAMIC0805-NOOUTLINE
- added D5: RED, SparkFun-LED:LED-RED1206
- added D6: GREEN, SparkFun-LED:LED-GREEN1206
- added Q2, Q3: 600mA/40V, SparkFun-DiscreteSemi:TRANS_NPN-MMBT2222AL
- added R24, R25: ???, microbuilder:RESISTOR0805
- added R26: 10K, adafruit:R-US_R0805
- added U6: CP2104, microbuilder:CP2104
- R8: value 0K -> 4.7K
- R9: value 0K -> 10K; device microbuilder:RESISTOR0805 -> adafruit:R-US_R0805
Connections:
- removed net CTS0: R6(NC).2
- removed net FTDI_CTS: J3.5, R6(NC).1
- removed net FTDI_RTS: J3.1, R12(NC).1
- removed net FTDI_RXD: J3.2, R9.1
- removed net FTDI_TXD: J3.3, R8.1
- removed net FTDI_VCC: J3.4
- removed net RTS0: R12(NC).2
- new net DTR: U6G$1.DTR
- new net IO0: U2.IO0
- new net N$36: JP9.D-, U6G$1.D-
- new net N$37: JP9.D+, U6G$1.D+
- new net N$39: U6G$1.TXD
- new net N$40: U6G$1.RXD
- new net N$41: D5.A, R24.2
- new net N$42: R24.1, U6G$1.GPIO0/TXLED
- new net N$43: R25.1, U6G$1.GPIO1/RXLED
- new net N$44: D6.A, R25.2
- new net N$46: Q3.C
- new net N$47: Q2.C
- new net N$48: R9.1
- new net N$49: R26.1
- new net RTS: U6G$1.RTS
- net GND: now also C11.2, C9.1, D5.C, D6.C, U6G$1.GND; no longer C7.2, J3.6
- net N$10: now also C9.2, U6G$1.VPP; no longer U2.TXD0
- net N$11: now also R8.2, U6G$1.#RST; no longer U2.RXD0
- net N$13: now also Q2.E, Q3.B, R9.2; no longer U2.IO22
- net N$14: now also Q2.B, Q3.E, R26.2; no longer U2.IO19
- net N$35: now also R22.1, R23.1, S2.1, S3.1
- net RXD0: now also U2.RXD0; no longer R8.2
- net TXD0: now also U2.TXD0; no longer R9.2
- net VCC: now also R8.1, U6G$1.VDD, U6G$1.VIO
- net VCC_3.7V: now also C11.1; no longer C7.1
- net VIN: now also U6G$1.REGIN, U6G$1.VBUS
Other:
- note removed: "FTDI MALE HEADER"
- note removed: "Is the logic levels correct on these? Maybe i should buy a different FTDI Cable"
- note removed: "Maybe add through hole to enable changing lipo, though i doubt we ever will."
- note removed: "REPLACE ALL 0604 with 0805"
- note removed: "https://www.adafruit.com/products/70"
- moved on the sheet: R13, R22, R23, R8, S1, S2, S3

Commit message: Reset and Bootloader PushButtons, Replaced USB
USB micro to mini due to supply issues.
SMD Xbee headers
New voltage regulator
Parts:
- removed JP9: Micro USB, SparkFun-Connectors:USB-ABCONN-11794
- removed U7: V_REG_317SMD, SparkFun-IC-Power:V_REG_317SMD
- added J1, J2: (no value), SparkFun-Connectors:CONN_102MMSMD
- added J4: USB_MINI-B_SMT, SparkFun-Connectors:USB_MINI-B_SMT
- added R27: 165, microbuilder:RESISTOR0805
- added S4, S5: MOMENTARY-SWITCH-SPST-SMD-6.0X3.5MM, SparkFun-Switches:MOMENTARY-SWITCH-SPST-SMD-6.0X3.5MM
- added U8: 3.3V, SparkFun-IC-Power:V_REG_AP2112K-3.3V
- R14: value ??? -> 2k
- R15: value 370 -> 10K; device microbuilder:RESISTOR0805 -> adafruit:R-US_R0805
- R16: value 220 -> 10K; device microbuilder:RESISTOR0805 -> adafruit:R-US_R0805
- R20: value ??? -> 20
- R6: value 0K -> 10K
- S1, S2, S3: value MOMENTARY-SWITCH-SPST-SMD-5.2MM -> MOMENTARY-SWITCH-SPST-SMD-6.0X3.5MM; device SparkFun-Switches:MOMENTARY-SWITCH-SPST-SMD-5.2MM -> SparkFun-Switches:MOMENTARY-SWITCH-SPST-SMD-6.0X3.5MM
Connections:
- net IO23 renamed IO26
- removed net +3V3: C2.1, U3.VDD
- new net N$38: R16.2, S5.2
- net CTS1: now also J1.9
- net GND: now also J2.10, J4.GND, R27.2, S4.1, S5.1, U8.GND; no longer JP9.GND, R15.1
- net IO7: now also J2.5
- net IO8: now also J2.9
- net N$24: now also S4.2; no longer R16.2, U7.ADJ
- net N$34: now also R27.1
- net N$36: now also J4.D-; no longer JP9.D-
- net N$37: now also J4.D+; no longer JP9.D+
- net RTS1: now also J1.5
- net RXD1: now also J2.2
- net TXD1: now also J2.3
- net VCC: now also C2.1, R15.1, U3.VDD, U8.OUT; no longer U7.OUT
- net VCC_3.7V: now also J2.1, U8.EN, U8.IN; no longer U7.IN
- net VIN: now also J4.VBUS; no longer JP9.VBUS
Other:
- note added: "Removal of R14 will reduce the charging circuit to 500mA"
- note added: "Set for 1000mA charging"
- note removed: "Set for 500mA charging"
- moved on the sheet: C1, C3, C4, C5, D1, D2, D3, FB3, FB4, Q1, Q2, Q3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

Commit message: Created Android Wear App
Sets the smart watch's bluetooth to discoverable.
Connections:
- net VIN renamed VBUS
Other:
- moved on the sheet: D1, D2, D3, R15, R17, R18, R19, S4
Changed lines of the file:
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@@
 <instance part="BT1" gate="G$1" x="228.6" y="147.32"/>
 <instance part="P+8" gate="VCC" x="236.22" y="109.22" rot="R180"/>
-<instance part="D1" gate="G$1" x="386.08" y="81.28" rot="R90"/>
-<instance part="D2" gate="G$1" x="386.08" y="68.58" rot="R90"/>
-<instance part="D3" gate="G$1" x="386.08" y="93.98" rot="R90"/>
-<instance part="R17" gate="G$1" x="375.92" y="81.28"/>
-<instance part="U$20" gate="G$1" x="408.94" y="60.96"/>
-<instance part="R18" gate="G$1" x="375.92" y="93.98"/>
-<instance part="R19" gate="G$1" x="375.92" y="68.58"/>
+<instance part="D1" gate="G$1" x="414.02" y="78.74" rot="R90"/>
+<instance part="D2" gate="G$1" x="414.02" y="66.04" rot="R90"/>
+<instance part="D3" gate="G$1" x="414.02" y="91.44" rot="R90"/>
+<instance part="R17" gate="G$1" x="403.86" y="78.74"/>
+<instance part="U$20" gate="G$1" x="436.88" y="58.42"/>
+<instance part="R18" gate="G$1" x="403.86" y="91.44"/>
+<instance part="R19" gate="G$1" x="403.86" y="66.04"/>
 <instance part="P+9" gate="VCC" x="363.22" y="139.7"/>
 <instance part="R20" gate="G$1" x="200.66" y="137.16" rot="R90"/>
@@
 <instance part="U8" gate="G$1" x="218.44" y="109.22"/>
 <instance part="GND6" gate="1" x="205.74" y="96.52"/>
-<instance part="R15" gate="G$1" x="111.76" y="-35.56" rot="R270"/>
-<instance part="U$22" gate="G$1" x="83.82" y="-55.88"/>
-<instance part="P+12" gate="VCC" x="111.76" y="-22.86"/>
+<instance part="R15" gate="G$1" x="109.22" y="-38.1" rot="R270"/>
+<instance part="U$22" gate="G$1" x="81.28" y="-58.42"/>
+<instance part="P+12" gate="VCC" x="109.22" y="-25.4"/>
 <instance part="R16" gate="G$1" x="109.22" y="-2.54" rot="R270"/>
 <instance part="U$23" gate="G$1" x="81.28" y="-22.86"/>
 <instance part="P+13" gate="VCC" x="109.22" y="10.16"/>
-<instance part="S4" gate="G$1" x="93.98" y="-45.72"/>
+<instance part="S4" gate="G$1" x="91.44" y="-48.26"/>
 <instance part="S5" gate="G$1" x="91.44" y="-12.7"/>
 <instance part="S1" gate="G$1" x="411.48" y="134.62"/>
@@
 <segment>
 <pinref part="U$20" gate="G$1" pin="GND"/>
-<wire x1="408.94" y1="63.5" x2="408.94" y2="68.58" width="0.1524" layer="91"/>
+<wire x1="436.88" y1="60.96" x2="436.88" y2="66.04" width="0.1524" layer="91"/>
 <pinref part="D1" gate="G$1" pin="C"/>
-<wire x1="408.94" y1="68.58" x2="408.94" y2="81.28" width="0.1524" layer="91"/>
-<wire x1="408.94" y1="81.28" x2="391.16" y2="81.28" width="0.1524" layer="91"/>
+<wire x1="436.88" y1="66.04" x2="436.88" y2="78.74" width="0.1524" layer="91"/>
+<wire x1="436.88" y1="78.74" x2="419.1" y2="78.74" width="0.1524" layer="91"/>
 <pinref part="D3" gate="G$1" pin="C"/>
-<wire x1="391.16" y1="93.98" x2="408.94" y2="93.98" width="0.1524" layer="91"/>
-<wire x1="408.94" y1="93.98" x2="408.94" y2="81.28" width="0.1524" layer="91"/>
+<wire x1="419.1" y1="91.44" x2="436.88" y2="91.44" width="0.1524" layer="91"/>
+<wire x1="436.88" y1="91.44" x2="436.88" y2="78.74" width="0.1524" layer="91"/>
 <pinref part="D2" gate="G$1" pin="C"/>
-<wire x1="391.16" y1="68.58" x2="408.94" y2="68.58" width="0.1524" layer="91"/>
-<junction x="408.94" y="68.58"/>
-<junction x="408.94" y="81.28"/>
+<wire x1="419.1" y1="66.04" x2="436.88" y2="66.04" width="0.1524" layer="91"/>
+<junction x="436.88" y="66.04"/>
+<junction x="436.88" y="78.74"/>
 </segment>
 <segment>
@@
 <segment>
 <pinref part="U$22" gate="G$1" pin="GND"/>
-<wire x1="83.82" y1="-53.34" x2="83.82" y2="-45.72" width="0.1524" layer="91"/>
-<wire x1="83.82" y1="-45.72" x2="88.9" y2="-45.72" width="0.1524" layer="91"/>
+<wire x1="81.28" y1="-55.88" x2="81.28" y2="-48.26" width="0.1524" layer="91"/>
+<wire x1="81.28" y1="-48.26" x2="86.36" y2="-48.26" width="0.1524" layer="91"/>
 <pinref part="S4" gate="G$1" pin="1"/>
 </segment>
@@
 <segment>
 <wire x1="182.88" y1="127" x2="190.5" y2="127" width="0.1524" layer="91"/>
-<wire x1="190.5" y1="127" x2="190.5" y2="116.84" width="0.1524" layer="91"/>
+<wire x1="190.5" y1="127" x2="190.5" y2="114.3" width="0.1524" layer="91"/>
 <pinref part="U4" gate="G$1" pin="PROG"/>
-<wire x1="190.5" y1="116.84" x2="182.88" y2="111.76" width="0.1524" layer="91"/>
-<wire x1="195.58" y1="111.76" x2="195.58" y2="116.84" width="0.1524" layer="91"/>
-<wire x1="195.58" y1="116.84" x2="190.5" y2="116.84" width="0.1524" layer="91"/>
-<junction x="190.5" y="116.84"/>
+<wire x1="195.58" y1="111.76" x2="195.58" y2="114.3" width="0.1524" layer="91"/>
+<wire x1="195.58" y1="114.3" x2="190.5" y2="114.3" width="0.1524" layer="91"/>
 <pinref part="R14" gate="G$1" pin="2"/>
+<wire x1="190.5" y1="114.3" x2="182.88" y2="114.3" width="0.1524" layer="91"/>
 <pinref part="R12" gate="G$1" pin="2"/>
+<wire x1="182.88" y1="114.3" x2="182.88" y2="111.76" width="0.1524" layer="91"/>
+<junction x="190.5" y="114.3"/>
 </segment>
 </net>
@@
 </segment>
 </net>
-<net name="VIN" class="0">
+<net name="VBUS" class="0">
 <segment>
 <wire x1="160.02" y1="101.6" x2="160.02" y2="99.06" width="0.1524" layer="91"/>
@@
 <pinref part="R22" gate="G$1" pin="2"/>
 <pinref part="R23" gate="G$1" pin="2"/>
+<junction x="363.22" y="134.62"/>
+<junction x="363.22" y="121.92"/>
 </segment>
 <segment>
@@
 <pinref part="R15" gate="G$1" pin="1"/>
 <pinref part="P+12" gate="VCC" pin="VCC"/>
-<wire x1="111.76" y1="-30.48" x2="111.76" y2="-25.4" width="0.1524" layer="91"/>
+<wire x1="109.22" y1="-33.02" x2="109.22" y2="-27.94" width="0.1524" layer="91"/>
 </segment>
 <segment>
@@
 <pinref part="R18" gate="G$1" pin="2"/>
 <pinref part="D3" gate="G$1" pin="A"/>
-<wire x1="381" y1="93.98" x2="383.54" y2="93.98" width="0.1524" layer="91"/>
+<wire x1="408.94" y1="91.44" x2="411.48" y2="91.44" width="0.1524" layer="91"/>
 </segment>
 </net>
@@
 <pinref part="R17" gate="G$1" pin="2"/>
 <pinref part="D1" gate="G$1" pin="A"/>
-<wire x1="381" y1="81.28" x2="383.54" y2="81.28" width="0.1524" layer="91"/>
+<wire x1="408.94" y1="78.74" x2="411.48" y2="78.74" width="0.1524" layer="91"/>
 </segment>
 </net>
@@
 <pinref part="R19" gate="G$1" pin="2"/>
 <pinref part="D2" gate="G$1" pin="A"/>
-<wire x1="381" y1="68.58" x2="383.54" y2="68.58" width="0.1524" layer="91"/>
+<wire x1="408.94" y1="66.04" x2="411.48" y2="66.04" width="0.1524" layer="91"/>
 </segment>
 </net>
@@
 <segment>
 <pinref part="R18" gate="G$1" pin="1"/>
-<wire x1="370.84" y1="93.98" x2="355.6" y2="93.98" width="0.1524" layer="91"/>
+<wire x1="398.78" y1="91.44" x2="383.54" y2="91.44" width="0.1524" layer="91"/>
 </segment>
 </net>
@@
 <segment>
 <pinref part="R17" gate="G$1" pin="1"/>
-<wire x1="370.84" y1="81.28" x2="355.6" y2="81.28" width="0.1524" layer="91"/>
+<wire x1="398.78" y1="78.74" x2="383.54" y2="78.74" width="0.1524" layer="91"/>
 </segment>
 </net>
@@
 <segment>
 <pinref part="R19" gate="G$1" pin="1"/>
-<wire x1="370.84" y1="68.58" x2="355.6" y2="68.58" width="0.1524" layer="91"/>
+<wire x1="398.78" y1="66.04" x2="383.54" y2="66.04" width="0.1524" layer="91"/>
 </segment>
 </net>
@@
 <label x="266.7" y="35.56" size="1.778" layer="95"/>
 <label x="266.7" y="35.56" size="1.778" layer="95"/>
-<label x="358.14" y="68.58" size="1.778" layer="95"/>
+<label x="386.08" y="66.04" size="1.778" layer="95"/>
 </segment>
 </net>
@@
 <label x="266.7" y="38.1" size="1.778" layer="95"/>
 <wire x1="279.4" y1="38.1" x2="264.16" y2="38.1" width="0.1524" layer="91"/>
-<label x="358.14" y="81.28" size="1.778" layer="95"/>
+<label x="386.08" y="78.74" size="1.778" layer="95"/>
 </segment>
 </net>
@@
 <wire x1="279.4" y1="40.64" x2="264.16" y2="40.64" width="0.1524" layer="91"/>
 <label x="266.7" y="40.64" size="1.778" layer="95"/>
-<label x="358.14" y="93.98" size="1.778" layer="95"/>
+<label x="386.08" y="91.44" size="1.778" layer="95"/>
 </segment>
 </net>
@@
 <label x="335.28" y="35.56" size="1.778" layer="95"/>
 <label x="114.3" y="17.78" size="1.778" layer="95" rot="MR0"/>
-<label x="127" y="-45.72" size="1.778" layer="95" rot="MR0"/>
+<label x="124.46" y="-48.26" size="1.778" layer="95" rot="MR0"/>
 </segment>
 </net>
@@
 <net name="N$24" class="0">
 <segment>
-<wire x1="99.06" y1="-45.72" x2="111.76" y2="-45.72" width="0.1524" layer="91"/>
+<wire x1="96.52" y1="-48.26" x2="109.22" y2="-48.26" width="0.1524" layer="91"/>
 <pinref part="R15" gate="G$1" pin="2"/>
-<wire x1="111.76" y1="-45.72" x2="129.54" y2="-45.72" width="0.1524" layer="91"/>
-<wire x1="111.76" y1="-40.64" x2="111.76" y2="-45.72" width="0.1524" layer="91"/>
-<junction x="111.76" y="-45.72"/>
+<wire x1="109.22" y1="-48.26" x2="127" y2="-48.26" width="0.1524" layer="91"/>
+<wire x1="109.22" y1="-43.18" x2="109.22" y2="-48.26" width="0.1524" layer="91"/>
+<junction x="109.22" y="-48.26"/>
 <pinref part="S4" gate="G$1" pin="2"/>
 </segment>

Commit message: Fixed Net Issues, Started Routing
Parts:
- added FRAME1: FRAME-LEDGER, SparkFun-Aesthetics:FRAME-LEDGER
- added LOGO1: OSHW-LOGOM, SparkFun-Aesthetics:OSHW-LOGOM
- added R28(NC), R29(NC): 0k, adafruit:R-US_R0805
Connections:
- removed net N$1: U2.SD2
- removed net N$12: U2.SD3
- removed net N$15: C6.2, R6.1
- removed net N$17: U2.SDO
- removed net N$18: U2.SD1
- removed net N$19: U2.IO17
- removed net N$2: U3.SCL
- removed net N$20: U2.IO34
- removed net N$21: U2.IO35
- removed net N$22: U2.IO16
- removed net N$24: R15.2, S4.2
- removed net N$28: R18.1
- removed net N$29: R17.1
- removed net N$30: R19.1
- removed net N$31: S1.2
- removed net N$32: S2.2
- removed net N$33: S3.2
- removed net N$34: R20.2, R27.1
- removed net N$38: R16.2, S5.2
- removed net N$39: U6G$1.TXD
- removed net N$4: U3.SDA
- removed net N$40: U6G$1.RXD
- removed net N$46: Q3.C
- removed net N$47: Q2.C
- removed net N$48: R9.1
- removed net N$49: R26.1
- removed net N$6: U2.CMD
- new net CTS: R28(NC).1, U6G$1.CTS
- new net IO13: R29(NC).2, U2.IO13
- new net IO15: R28(NC).2, U2.IO15
- net DTR: now also R9.1
- net EN: now also C6.2, Q3.C, R16.2, R6.1, S5.2
- net IO0: now also Q2.C, R15.2, S4.2
- net IO12: now also R19.1
- net IO14: now also R17.1
- net IO25: now also S2.2
- net IO26: now also S3.2
- net IO27: now also R18.1
- net IO32: now also R20.2, R27.1
- net IO33: now also S1.2
- net IO34: now also U2.IO34
- net IO35: now also U2.IO35
- net IO8: now also U2.SD1, U2.SDO
- net RTS: now also R26.1, R29(NC).1, U6G$1.RXD
- net RTS1: now also U2.CMD
- net RXD0: now also U6G$1.TXD
- net RXD1: now also U2.SD2
- net SCL: now also U2.IO17, U3.SCL
- net SDA: now also U2.IO16, U3.SDA
- net TXD1: now also U2.SD3
Other:
- note added: "Brian Sheridan"
- moved on the sheet: C1, C10, C11, C2, C3, C4, C5, C6, C8, C9, D1, D2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
