File: PCB/SensorNode.sch (EAGLE design)
At the start: 72 parts, among them J4 USB_MINI-B_SMT, Q1 CMA-4544PF-W, Q2 600mA/40V, Q3 600mA/40V, U1 MAX4466EXK+T, U2 ESP-WROOM-32, U3 Si7021-A20, U4 MCP73831, U5 TSL2561, U6 CP2104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

Commit message: Mid Route Check Point
Parts:
- removed R16: 10K, adafruit:R-US_R0805
- removed U$1: XBEE, adafruit:XBEE
Connections:
- net CTS1: no longer U$1.CTS/DIO7
- net EN: no longer R16.2
- net GND: no longer U$1.GND
- net IO7: no longer U$1.RESET
- net IO8: no longer U$1.DTR/DI8
- net RTS1: no longer U$1.RTS/AD6/DIO6
- net RXD1: no longer U$1.DOUT
- net TXD1: no longer U$1.DIN
- net VCC: no longer R16.1
- net VCC_3.7V: no longer U$1.VCC
Other:
- moved on the sheet: C6, R15, R6, S4, S5
Changed lines of the file:
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@@
 <part name="P+7" library="microbuilder" deviceset="VCC" device=""/>
 <part name="U2" library="esp32" deviceset="ESP-WROOM-32" device=""/>
-<part name="U$1" library="adafruit" deviceset="XBEE" device=""/>
 <part name="U1" library="microbuilder" deviceset="MAX4466" device="&quot;&quot;" value="MAX4466EXK+T"/>
 <part name="FB3" library="microbuilder" deviceset="FERRITE" device="0805" value="FERRITE"/>
@@
 <part name="U$22" library="microbuilder" deviceset="GND" device=""/>
 <part name="P+12" library="microbuilder" deviceset="VCC" device=""/>
-<part name="R16" library="adafruit" deviceset="R-US_" device="R0805" value="10K"/>
 <part name="U$23" library="microbuilder" deviceset="GND" device=""/>
-<part name="P+13" library="microbuilder" deviceset="VCC" device=""/>
 <part name="S4" library="SparkFun-Switches" deviceset="MOMENTARY-SWITCH-SPST" device="-SMD-6.0X3.5MM"/>
 <part name="S5" library="SparkFun-Switches" deviceset="MOMENTARY-SWITCH-SPST" device="-SMD-6.0X3.5MM"/>
@@
 <instance part="P+7" gate="VCC" x="345.44" y="101.6"/>
 <instance part="U2" gate="G$1" x="256.54" y="170.18"/>
-<instance part="U$1" gate="G$1" x="373.38" y="132.08"/>
 <instance part="U1" gate="G$1" x="172.72" y="116.84"/>
 <instance part="FB3" gate="G$1" x="172.72" y="149.86"/>
@@
 <instance part="P+6" gate="VCC" x="223.52" y="177.8"/>
 <instance part="U$18" gate="G$1" x="294.64" y="177.8" rot="R180"/>
-<instance part="P+4" gate="VCC" x="213.36" y="254"/>
-<instance part="R6" gate="G$1" x="213.36" y="243.84" rot="R90"/>
-<instance part="C6" gate="G$1" x="213.36" y="220.98" rot="R180"/>
-<instance part="U$21" gate="G$1" x="213.36" y="205.74"/>
+<instance part="P+4" gate="VCC" x="58.42" y="71.12"/>
+<instance part="R6" gate="G$1" x="58.42" y="60.96" rot="R90"/>
+<instance part="C6" gate="G$1" x="58.42" y="38.1" rot="R180"/>
+<instance part="U$21" gate="G$1" x="58.42" y="22.86"/>
 <instance part="GND1" gate="1" x="193.04" y="228.6"/>
 <instance part="GND15" gate="1" x="22.86" y="215.9"/>
@@
 <instance part="U8" gate="G$1" x="177.8" y="213.36"/>
 <instance part="GND6" gate="1" x="165.1" y="200.66"/>
-<instance part="R15" gate="G$1" x="68.58" y="35.56" rot="R270"/>
-<instance part="U$22" gate="G$1" x="40.64" y="15.24"/>
-<instance part="P+12" gate="VCC" x="68.58" y="48.26"/>
-<instance part="R16" gate="G$1" x="68.58" y="71.12" rot="R270"/>
-<instance part="U$23" gate="G$1" x="40.64" y="50.8"/>
-<instance part="P+13" gate="VCC" x="68.58" y="83.82"/>
-<instance part="S4" gate="G$1" x="50.8" y="25.4"/>
-<instance part="S5" gate="G$1" x="50.8" y="60.96"/>
+<instance part="R15" gate="G$1" x="129.54" y="43.18" rot="R270"/>
+<instance part="U$22" gate="G$1" x="101.6" y="22.86"/>
+<instance part="P+12" gate="VCC" x="129.54" y="55.88"/>
+<instance part="U$23" gate="G$1" x="27.94" y="38.1"/>
+<instance part="S4" gate="G$1" x="111.76" y="33.02"/>
+<instance part="S5" gate="G$1" x="38.1" y="48.26"/>
 <instance part="S1" gate="G$1" x="370.84" y="238.76"/>
 <instance part="S2" gate="G$1" x="370.84" y="226.06"/>
@@
 <pinref part="U$6" gate="G$1" pin="GND"/>
 <wire x1="345.44" y1="114.3" x2="345.44" y2="119.38" width="0.1524" layer="91"/>
-<pinref part="U$1" gate="G$1" pin="GND"/>
 <wire x1="345.44" y1="119.38" x2="350.52" y2="119.38" width="0.1524" layer="91"/>
 <pinref part="J2" gate="G$1" pin="10"/>
@@
 <pinref part="U$21" gate="G$1" pin="GND"/>
 <pinref part="C6" gate="G$1" pin="1"/>
-<wire x1="213.36" y1="208.28" x2="213.36" y2="215.9" width="0.1524" layer="91"/>
+<wire x1="58.42" y1="25.4" x2="58.42" y2="33.02" width="0.1524" layer="91"/>
 </segment>
 <segment>
@@
 <segment>
 <pinref part="U$22" gate="G$1" pin="GND"/>
-<wire x1="40.64" y1="17.78" x2="40.64" y2="25.4" width="0.1524" layer="91"/>
-<wire x1="40.64" y1="25.4" x2="45.72" y2="25.4" width="0.1524" layer="91"/>
+<wire x1="101.6" y1="25.4" x2="101.6" y2="33.02" width="0.1524" layer="91"/>
+<wire x1="101.6" y1="33.02" x2="106.68" y2="33.02" width="0.1524" layer="91"/>
 <pinref part="S4" gate="G$1" pin="1"/>
 </segment>
 <segment>
 <pinref part="U$23" gate="G$1" pin="GND"/>
-<wire x1="40.64" y1="53.34" x2="40.64" y2="60.96" width="0.1524" layer="91"/>
-<wire x1="40.64" y1="60.96" x2="45.72" y2="60.96" width="0.1524" layer="91"/>
+<wire x1="27.94" y1="40.64" x2="27.94" y2="48.26" width="0.1524" layer="91"/>
+<wire x1="27.94" y1="48.26" x2="33.02" y2="48.26" width="0.1524" layer="91"/>
 <pinref part="S5" gate="G$1" pin="1"/>
 </segment>
@@
 <pinref part="P+3" gate="VCC" pin="VCC"/>
 <wire x1="345.44" y1="149.86" x2="345.44" y2="142.24" width="0.1524" layer="91"/>
-<pinref part="U$1" gate="G$1" pin="VCC"/>
 <wire x1="345.44" y1="142.24" x2="350.52" y2="142.24" width="0.1524" layer="91"/>
 <pinref part="J2" gate="G$1" pin="1"/>
@@
 <pinref part="R6" gate="G$1" pin="2"/>
 <pinref part="P+4" gate="VCC" pin="VCC"/>
-<wire x1="213.36" y1="248.92" x2="213.36" y2="251.46" width="0.1524" layer="91"/>
+<wire x1="58.42" y1="66.04" x2="58.42" y2="68.58" width="0.1524" layer="91"/>
 </segment>
 <segment>
@@
 <net name="TXD1" class="0">
 <segment>
-<pinref part="U$1" gate="G$1" pin="DIN"/>
 <label x="337.82" y="137.16" size="1.778" layer="95"/>
 <label x="259.08" y="116.84" size="1.778" layer="95" rot="R90"/>
@@
 <pinref part="R6" gate="G$1" pin="1"/>
 <pinref part="C6" gate="G$1" pin="2"/>
-<wire x1="213.36" y1="238.76" x2="213.36" y2="231.14" width="0.1524" layer="91"/>
-<wire x1="213.36" y1="231.14" x2="213.36" y2="223.52" width="0.1524" layer="91"/>
-<wire x1="213.36" y1="231.14" x2="228.6" y2="231.14" width="0.1524" layer="91"/>
-<junction x="213.36" y="231.14"/>
-<label x="223.52" y="231.14" size="1.778" layer="95"/>
-</segment>
-<segment>
-<wire x1="55.88" y1="60.96" x2="68.58" y2="60.96" width="0.1524" layer="91"/>
-<pinref part="R16" gate="G$1" pin="2"/>
-<wire x1="68.58" y1="60.96" x2="86.36" y2="60.96" width="0.1524" layer="91"/>
-<wire x1="68.58" y1="66.04" x2="68.58" y2="60.96" width="0.1524" layer="91"/>
-<junction x="68.58" y="60.96"/>
+<wire x1="58.42" y1="55.88" x2="58.42" y2="48.26" width="0.1524" layer="91"/>
+<wire x1="58.42" y1="48.26" x2="58.42" y2="40.64" width="0.1524" layer="91"/>
+<wire x1="58.42" y1="48.26" x2="73.66" y2="48.26" width="0.1524" layer="91"/>
+<junction x="58.42" y="48.26"/>
+<label x="68.58" y="48.26" size="1.778" layer="95"/>
 <pinref part="S5" gate="G$1" pin="2"/>
-<label x="78.74" y="60.96" size="1.778" layer="95"/>
+<wire x1="58.42" y1="48.26" x2="43.18" y2="48.26" width="0.2032" layer="91"/>
 </segment>
 <segment>
@@
 <net name="RXD1" class="0">
 <segment>
-<pinref part="U$1" gate="G$1" pin="DOUT"/>
 <wire x1="350.52" y1="139.7" x2="335.28" y2="139.7" width="0.1524" layer="91"/>
 <label x="337.82" y="139.7" size="1.778" layer="95"/>
@@
 <net name="IO7" class="0">
 <segment>
-<pinref part="U$1" gate="G$1" pin="RESET"/>
 <wire x1="350.52" y1="132.08" x2="335.28" y2="132.08" width="0.1524" layer="91"/>
 <label x="337.82" y="132.08" size="1.778" layer="95"/>
@@
 <net name="CTS1" class="0">
 <segment>
-<pinref part="U$1" gate="G$1" pin="CTS/DIO7"/>
 <wire x1="398.78" y1="121.92" x2="416.56" y2="121.92" width="0.1524" layer="91"/>
 <label x="408.94" y="121.92" size="1.778" layer="95"/>
@@
 <net name="IO8" class="0">
 <segment>
-<pinref part="U$1" gate="G$1" pin="DTR/DI8"/>
 <wire x1="350.52" y1="121.92" x2="335.28" y2="121.92" width="0.1524" layer="91"/>
 <label x="337.82" y="121.92" size="1.778" layer="95"/>
@@
 <net name="RTS1" class="0">
 <segment>
-<pinref part="U$1" gate="G$1" pin="RTS/AD6/DIO6"/>
 <wire x1="398.78" y1="132.08" x2="416.56" y2="132.08" width="0.1524" layer="91"/>
 <label x="408.94" y="132.08" size="1.778" layer="95"/>
@@
 <pinref part="R15" gate="G$1" pin="1"/>
 <pinref part="P+12" gate="VCC" pin="VCC"/>
-<wire x1="68.58" y1="40.64" x2="68.58" y2="45.72" width="0.1524" layer="91"/>
-</segment>
-<segment>
-<pinref part="R16" gate="G$1" pin="1"/>
-<pinref part="P+13" gate="VCC" pin="VCC"/>
-<wire x1="68.58" y1="76.2" x2="68.58" y2="81.28" width="0.1524" layer="91"/>
+<wire x1="129.54" y1="48.26" x2="129.54" y2="53.34" width="0.1524" layer="91"/>
 </segment>
 <segment>
@@
 </segment>
 <segment>
-<wire x1="55.88" y1="25.4" x2="68.58" y2="25.4" width="0.1524" layer="91"/>
+<wire x1="116.84" y1="33.02" x2="129.54" y2="33.02" width="0.1524" layer="91"/>
 <pinref part="R15" gate="G$1" pin="2"/>
-<wire x1="68.58" y1="25.4" x2="86.36" y2="25.4" width="0.1524" layer="91"/>
-<wire x1="68.58" y1="30.48" x2="68.58" y2="25.4" width="0.1524" layer="91"/>
-<junction x="68.58" y="25.4"/>
+<wire x1="129.54" y1="33.02" x2="147.32" y2="33.02" width="0.1524" layer="91"/>
+<wire x1="129.54" y1="38.1" x2="129.54" y2="33.02" width="0.1524" layer="91"/>
+<junction x="129.54" y="33.02"/>
 <pinref part="S4" gate="G$1" pin="2"/>
-<label x="78.74" y="25.4" size="1.778" layer="95"/>
-</segment>
-<segment>
+<label x="139.7" y="33.02" size="1.778" layer="95"/>
+</segment>
+<segment>

Commit message: Commit Before AutoRouting
Parts:
- removed C11: 0.1uF, microbuilder:CAP_CERAMIC0805-NOOUTLINE
- removed R28(NC), R29(NC): 0k, adafruit:R-US_R0805
Connections:
- removed net CTS: R28(NC).1, U6G$1.CTS
- removed net IO13: R29(NC).2, U2.IO13
- removed net IO15: R28(NC).2, U2.IO15
- removed net N$16: U2.CLK
- removed net N$35: R13.1, R22.1, R23.1, S1.1, S2.1, S3.1
- new net N$24: R13.1, S1.1
- new net N$28: R22.1, S2.1
- new net N$29: R23.1, S3.1
- new net N$32: C3.2, R1.2, R2.1
- net AGND: no longer C3.2, R1.2, R2.1
- net CTS1: now also U2.CLK
- net GND: no longer C11.2
- net IO7: now also U2.SDO
- net IO8: no longer U2.SDO
- net RTS: no longer R29(NC).1, U6G$1.RXD
- net TXD0: now also U6G$1.RXD
- net VCC: now also FB4.P$2, J2.1, JP1.1, R10.2, R11.2, R6.2, U2.3V3, U5.3.3V
- net VCC_3.7V: no longer C11.1, FB4.P$2, J2.1, JP1.1, R10.2, R11.2, R6.2, U2.3V3, U5.3.3V

Commit message: Fully Routed
Parts:
- removed BT1: LIPO-OUTLINE1100, SparkFun-Batteries:LIPO-OUTLINE1100
Changed lines of the file:
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@@
 <part name="GND19" library="SparkFun" deviceset="GND" device=""/>
 <part name="JP2" library="SparkFun-Connectors" deviceset="JST_2MM_MALE" device="" value="JST"/>
-<part name="BT1" library="SparkFun-Batteries" deviceset="LIPO-OUTLINE" device="1100"/>
 <part name="P+8" library="microbuilder" deviceset="VCC" device=""/>
 <part name="D1" library="SparkFun-LED" deviceset="LED-BLUE" device="1206" value="BLUE"/>
@@
 <instance part="GND19" gate="1" x="149.86" y="200.66"/>
 <instance part="JP2" gate="G$1" x="193.04" y="241.3" rot="MR0"/>
-<instance part="BT1" gate="G$1" x="187.96" y="251.46"/>
 <instance part="P+8" gate="VCC" x="195.58" y="213.36" rot="R180"/>
 <instance part="D1" gate="G$1" x="373.38" y="182.88" rot="R90"/>
