File: PCB/SensorNode.brd (EAGLE design)
At the start: 58.9 x 70.1 mm, 66 parts, among them J4 USB_MINI-B_SMT, Q1 CMA-4544PF-W, Q2 600mA/40V, Q3 600mA/40V, U1 MAX4466EXK+T, U2 ESP-WROOM-32, U3 Si7021-A20, U4 MCP73831, U5 TSL2561, U6 CP2104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

Commit message: Post DRC layout
Parts:
- moved R2 0.30 mm to (42.3, 24.9)
- moved S1 0.30 mm to (12.9, 52.1)
- moved R8 0.25 mm to (14.5, 2.88)
Routing:
- net GND: track 322.4 -> 300.2 mm, vias 8 -> 7
- net N$18: track 5.84 -> 0.00 mm
- net VBUS: track 36.6 -> 38.0 mm
- net N$43: track 5.74 -> 6.39 mm
- net N$20: track 0.61 -> 0.00 mm
- net SCL: track 24.4 -> 25.0 mm
- added copper zone on layer 16, net GND
Other:
- board text added: "Corvus Perception SensorNode V1"
